File: drone-fc/kicad/drone-fc.kicad_pcb (KiCad board)
At the start: 4 copper layers, 45 x 45 mm, 83 parts, among them J4 Conn_01x01_Pin, U1 TPS62177DQC, U2 STM32F407VETx, U3 LSM6DSM, U6 BMP581, U8 TPS62175DQC, Y1 Crystal_GND24

Commit message: Replaced BMP581 with BMP388
Parts:
- removed U6: BMP581, BMP581:BMP581
- added U5: BMP388, BMP388:BMP388, F.Cu at (205.0, 96.2)
